File: Hardware/TGO.brd (EAGLE design)
At the start: 25.4 x 25.4 mm, 45 parts, among them J4 SMD_PAD, U1 AP3012, U2 SAS1-1U001-A_I2C_4WSPI

Commit message: Finish prototype v01
Parts:
- removed LOGO1: SFE_LOGO_NAME_FLAME.1_INCH, SparkFun-Aesthetics:SFE_LOGO_NAME_FLAME_.1
- added U$14: (no value), buzzard_labels:GND0
- added U$15: (no value), buzzard_labels:D##C6
- added U$16: (no value), buzzard_labels:GND10
- added U$17: (no value), buzzard_labels:3V311
- added U$18: (no value), buzzard_labels:013
- added U$19: (no value), buzzard_labels:112
- added U$20: (no value), buzzard_labels:4WSPI14
- added U$21, U$22: (no value), buzzard_labels:I2C13
- added U$23: (no value), SparkFun-Aesthetics:SFE_LOGO_NAME_.1
- added U$24: (no value), SparkFun-Aesthetics:SFE_LOGO_FLAME_.1
- added U$25: (no value), buzzard_labels:#CS#PULL19
- added U$26: (no value), buzzard_labels:IFS17
- added U$27: (no value), buzzard_labels:D2#SDA19
- U$10: device buzzard_labels:#CS7 -> buzzard_labels:MOSI9
- U$11: device buzzard_labels:#CS6 -> buzzard_labels:SCLK8
- U$13: device buzzard_labels:D##C9 -> buzzard_labels:3V31
- U$2: device Labels:QWIIC_COPYRIGHT_SMALL -> buzzard_labels:QWIIC_TRANSPARENT_GRAPHICAL_OLED15
- U$3: device Labels:QWIIC_COPYRIGHT_SMALL -> buzzard_labels:SA0_PULL19
- U$8: device buzzard_labels:SCLK4 -> buzzard_labels:#CS7
- U$9: device buzzard_labels:MOSI5 -> buzzard_labels:NC10
- moved FRAME1 74.5 mm to (-11.4, -10.2)
- moved LOGO2 62.8 mm to (3.17, 18.3)
- moved U$2 45.2 mm to (25.7, 19.7), flipped to the bottom
- moved U$3 34.9 mm to (15.2, 11.0), flipped to the bottom, turned to 90 degrees
- moved U$13 11.0 mm to (8.89, 1.40), turned to 90 degrees
- moved U$8 7.46 mm to (16.5, 1.27), turned to 90 degrees
- moved U$11 6.20 mm to (11.4, 1.40), turned to 90 degrees
- moved U$9 5.91 mm to (16.5, 1.40), turned to 90 degrees
- moved U$10 2.54 mm to (14.0, 1.40), flipped to the bottom
- moved JP1 1.27 mm to (20.3, 7.62)
- moved JP2 1.27 mm to (15.2, 7.62)
- moved JP3 1.27 mm to (10.2, 7.62)
- moved JP4 1.27 mm to (5.08, 7.62)
Routing:
- net 3.3V: track 65.0 -> 69.7 mm
- net NC/D2: track 20.3 -> 24.5 mm
- net N$2: track 7.40 -> 5.54 mm
- net D!C!/SA0: track 33.5 -> 31.8 mm
- net N$7: track 3.71 -> 5.11 mm
- net N$6: track 12.2 -> 13.4 mm
- net !CS: track 25.9 -> 27.0 mm
- net 12V: track 34.3 -> 33.3 mm
- net !RES: track 27.3 -> 26.2 mm
- net N$1: track 20.9 -> 20.0 mm
- net GND: track 41.1 -> 41.0 mm, vias 18 -> 24
Other:
- board text added: "Owen Lyke"
- board text added: "v01"
