File: Hardware/TGO.brd (EAGLE design)
At the start: 25.4 x 25.4 mm, 59 parts, among them U1 AP3012, U2 SAS1-1U001-A_I2C_4WSPI

Commit message: Move display into SparkFun library
Parts:
- U2: value SAS1-1U001-A_I2C_4WSPI -> UG-2856KLBAG01_4WSPI; device TGO:FPC05024-42201 -> SparkFun-Displays:FPC05024-42201

Commit message: Add pullup resistors on I2C lines, increment version number
Parts:
- added R8, R9: 2.2k, SparkFun-Resistors:0603
Connections:
- net 3.3V: now also R8.2, R9.2
- net SCLK/SCL: now also R9.1
- net SDIN/SDA: now also R8.1
Other:
- board text added: "v02"
- board text removed: "v01"
Changed lines of the file:
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@@
 <setting verticaltext="up"/>
 </settings>
-<grid distance="0.005" unitdist="inch" unit="inch" style="lines" multiple="1" display="yes" altdistance="0.005" altunitdist="inch" altunit="inch"/>
+<grid distance="0.05" unitdist="inch" unit="inch" style="lines" multiple="1" display="yes" altdistance="0.005" altunitdist="inch" altunit="inch"/>
 <layers>
-<layer number="1" name="Top" color="4" fill="1" visible="no" active="yes"/>
-<layer number="16" name="Bottom" color="1" fill="1" visible="no" active="yes"/>
+<layer number="1" name="Top" color="4" fill="1" visible="yes" active="yes"/>
+<layer number="16" name="Bottom" color="1" fill="1" visible="yes" active="yes"/>
 <layer number="17" name="Pads" color="2" fill="1" visible="yes" active="yes"/>
-<layer number="18" name="Vias" color="2" fill="1" visible="no" active="yes"/>
-<layer number="19" name="Unrouted" color="6" fill="1" visible="no" active="yes"/>
+<layer number="18" name="Vias" color="2" fill="1" visible="yes" active="yes"/>
+<layer number="19" name="Unrouted" color="6" fill="1" visible="yes" active="yes"/>
 <layer number="20" name="Dimension" color="15" fill="1" visible="yes" active="yes"/>
 <layer number="21" name="tPlace" color="16" fill="1" visible="yes" active="yes"/>
-<layer number="22" name="bPlace" color="14" fill="1" visible="no" active="yes"/>
+<layer number="22" name="bPlace" color="14" fill="1" visible="yes" active="yes"/>
 <layer number="23" name="tOrigins" color="15" fill="1" visible="yes" active="yes"/>
-<layer number="24" name="bOrigins" color="15" fill="1" visible="no" active="yes"/>
+<layer number="24" name="bOrigins" color="15" fill="1" visible="yes" active="yes"/>
 <layer number="25" name="tNames" color="7" fill="1" visible="no" active="yes"/>
 <layer number="26" name="bNames" color="7" fill="1" visible="no" active="yes"/>
-<layer number="27" name="tValues" color="7" fill="1" visible="yes" active="yes"/>
+<layer number="27" name="tValues" color="7" fill="1" visible="no" active="yes"/>
 <layer number="28" name="bValues" color="7" fill="1" visible="no" active="yes"/>
 <layer number="29" name="tStop" color="7" fill="3" visible="no" active="yes"/>
 <layer number="30" name="bStop" color="7" fill="6" visible="no" active="yes"/>
-<layer number="31" name="tCream" color="7" fill="4" visible="yes" active="yes"/>
+<layer number="31" name="tCream" color="7" fill="4" visible="no" active="yes"/>
 <layer number="32" name="bCream" color="7" fill="5" visible="no" active="yes"/>
 <layer number="33" name="tFinish" color="6" fill="3" visible="no" active="yes"/>
@@
 <wire x1="25.4" y1="25.4" x2="0" y2="25.4" width="0.2032" layer="20"/>
 <wire x1="0" y1="25.4" x2="0" y2="0" width="0.2032" layer="20"/>
-<text x="0.381" y="10.668" size="1.778" layer="16" font="vector" ratio="15" rot="SMR90">v01</text>
+<text x="0.381" y="10.668" size="1.778" layer="16" font="vector" ratio="15" rot="SMR90">v02</text>
 <text x="16.51" y="-10.16" size="1.778" layer="51" font="vector" ratio="15">Owen Lyke</text>
 <wire x1="2.413" y1="20.32" x2="1.27" y2="19.177" width="0.2032" layer="49"/>
@@
 <element name="FRAME1" library="SparkFun-Aesthetics" package="CREATIVE_COMMONS" value="FRAME-LETTER" x="-11.43" y="-10.16">
 <attribute name="DESIGNER" value="Owen Lyke" x="-11.43" y="-10.16" size="1.778" layer="27" display="off"/>
-<attribute name="REV" value="v01" x="-11.43" y="-10.16" size="1.778" layer="27" display="off"/>
+<attribute name="REV" value="v02" x="-11.43" y="-10.16" size="1.778" layer="27" display="off"/>
 </element>
 <element name="J1" library="SparkFun-Connectors" package="1X04_1MM_RA" value="" x="20.32" y="12.7" smashed="yes" rot="R90">
@@
 <element name="U$3" library="buzzard_labels_1" package="D27" value="" x="5.08" y="13.97" rot="MR90"/>
 <element name="U$20" library="buzzard_labels_1" package="D27" value="" x="10.16" y="13.97" rot="MR90"/>
+<element name="R8" library="SparkFun-Resistors" package="0603" value="2.2k" x="-30.48" y="-13.97">
+<attribute name="PROD_ID" value="RES-08272" x="-30.48" y="-13.97" size="1.778" layer="27" font="vector" ratio="15" display="off"/>
+</element>
+<element name="R9" library="SparkFun-Resistors" package="0603" value="2.2k" x="-30.48" y="-17.78">
+<attribute name="PROD_ID" value="RES-08272" x="-30.48" y="-17.78" size="1.778" layer="27" font="vector" ratio="15" display="off"/>
+</element>
 </elements>
 <signals>
@@
 <wire x1="14.859" y1="6.262" x2="17.018" y2="6.262" width="0.508" layer="1"/>
 <wire x1="17.018" y1="5.207" x2="16.256" y2="4.445" width="0.508" layer="1"/>
+<contactref element="R8" pad="2"/>
+<contactref element="R9" pad="2"/>
+<wire x1="-29.63" y1="-13.97" x2="-29.63" y2="-17.78" width="0" layer="19" extent="1-1"/>
+<wire x1="8.89" y1="1.27" x2="-29.63" y2="-13.97" width="0" layer="19" extent="1-1"/>
 </signal>
 <signal name="12V">
@@
 <wire x1="12.367259375" y1="11.02868125" x2="12.773" y2="10.622940625" width="0.2032" layer="1"/>
 <wire x1="12.773" y1="10.622940625" x2="12.773" y2="10.32025" width="0.2032" layer="1"/>
+<contactref element="R9" pad="1"/>
+<wire x1="4.064" y1="4.826" x2="-31.33" y2="-17.78" width="0" layer="19" extent="1-1"/>
 </signal>
 <signal name="SDIN/SDA">
@@
 <wire x1="11.77035" y1="10.45895" x2="11.77035" y2="12.53235" width="0.2032" layer="16"/>
 <wire x1="11.91768125" y1="10.31161875" x2="11.79068125" y2="10.18461875" width="0.2032" layer="1"/>
+<contactref element="R8" pad="1"/>
+<wire x1="4.572" y1="5.461" x2="-31.33" y2="-13.97" width="0" layer="19" extent="1-16"/>
 </signal>
 <signal name="D!C!/SA0">
