File: Hardware/SparkFun_Transparent_Graphical_OLED_Breakout.sch (EAGLE design)
At the start: 44 parts, among them U1 AP3012, U2 UG-2856KLBAG01_4WSPI

Commit message: Add External Display Indicator to help avoid BOM issues
Parts:
- added U$26: EXTERNAL_DISP-UG-2856KLBAG01, SparkFun-Displays:EXTERNAL_DISP-UG-2856KLBAG01
Changed lines of the file:
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@@
 <part name="H4" library="SparkFun-Hardware" deviceset="STAND-OFF" device=""/>
 <part name="TP1" library="SparkFun-Connectors" deviceset="TEST-POINT" device="3" value="12V"/>
+<part name="U$26" library="SparkFun-Displays" deviceset="EXTERNAL_DISP" device="-UG-2856KLBAG01"/>
 </parts>
 <sheets>
@@
 <attribute name="VALUE" x="139.7" y="93.98" size="1.778" layer="96" font="vector"/>
 </instance>
+<instance part="U$26" gate="G$1" x="78.74" y="124.46"/>
 </instances>
 <busses>
